File: adc_7seg_v0.kicad_pcb (KiCad board)
At the start: 4 copper layers, 34 parts, among them J1 IN, J2 DC, Q1 BC847, U1 MC78M09C, U2 ICL7106, U3 TDSR1350, U4 TDSR1350, U5 TDSR1350

Commit message: last version, too big
Parts:
- added H1: Bolt, KLALIB_Mechanical:Bolt_M3, F.Cu at (163.2, 100.3)
- added H2: Bolt, KLALIB_Mechanical:Bolt_M3, F.Cu at (232.4, 100.3)
- added H3: Bolt, KLALIB_Mechanical:Bolt_M3, F.Cu at (163.2, 80.6)
- added H4: Bolt, KLALIB_Mechanical:Bolt_M3, F.Cu at (232.4, 80.6)
- moved C4 11.0 mm to (216.8, 81.0), turned to 180 degrees
- moved C3 4.68 mm to (212.6, 80.3), turned to 270 degrees
- moved R13 0.85 mm to (217.7, 85.1), turned to 180 degrees
- moved R12 0.38 mm to (188.3, 102.7)
Routing:
- net GND: track 0.00 -> 27.8 mm, vias 0 -> 68
- net Net-(C1-Pad1): track 0.00 -> 12.6 mm
- net Net-(U2-Pad32): track 47.0 -> 42.9 mm
- net Net-(U2-Pad30): track 50.9 -> 48.5 mm
- net Net-(U2-Pad29): track 57.6 -> 55.6 mm
- net Net-(U3-Pad8): track 31.0 -> 29.8 mm
- net Net-(U2-Pad25): track 46.2 -> 47.3 mm
- net Net-(JP4-Pad3): track 7.12 -> 6.59 mm
- net Net-(Q1-Pad1): track 13.6 -> 13.8 mm, vias 2 -> 1
- net +9V: track 84.2 -> 84.3 mm, vias 2 -> 1
- added copper zone on B.Cu, net GND
- added copper zone on F.Cu, net GND
Other:
- board outline added: 75.4 x 26.2 mm
- copper layers 4 -> 2
- net class Default: clearance 0.2 -> 0.1524
- rule trace_clearance: 0.2 -> 0.1524
- rule via_min_size: 0.4 -> 0.3
