File: adc_7seg_v0.sch (KiCad schematic (older format))
At the start: 34 parts, among them J1 IN, J2 DC, Q1 BC847, U1 MC78M09C, U2 ICL7106, U3 TDSR1350, U4 TDSR1350, U5 TDSR1350

Commit message: last good version, skoro naroutovana
Parts:
- C4: footprint Capacitor_THT:CP_Radial_D8.0mm_P3.50mm -> Capacitor_THT:CP_Radial_D6.3mm_P2.50mm
Connections:
- net at Q1.2 (E), U5.3 (CA): no longer U3.3 (CA), U4.3 (CA)
- net at U3.8 (CA): now also U4.8 (CA), U5.8 (CA)
- no-connect marks 3 -> 6
Changed lines of the file:
@@
 Wire Wire Line
 	5700 5200 6550 5200
-Wire Wire Line
-	6350 1950 6350 1800
 $Comp
 L Device:R R13
@@
 	1    0    0    -1
 $EndComp
-Wire Wire Line
-	7400 1950 7400 1800
-Wire Wire Line
-	8450 1950 8450 1800
 $Comp
 L KLALIB_Analog_ADC:ICL7106 U2
@@
 	3250 3450 3400 3450
 Wire Wire Line
-	6350 1800 7400 1800
-Wire Wire Line
-	8450 1800 7400 1800
-Connection ~ 7400 1800
-Wire Wire Line
-	8450 1800 9050 1800
-Wire Wire Line
 	9050 1800 9050 5900
 Wire Wire Line
 	9050 5900 6250 5900
-Connection ~ 8450 1800
 NoConn ~ 5700 5300
 NoConn ~ 5700 5400
@@
 F 0 "C4" H 5018 2746 50  0000 L CNN
 F 1 "100u" H 5018 2655 50  0000 L CNN
-F 2 "Capacitor_THT:CP_Radial_D8.0mm_P3.50mm" H 4938 2550 50  0001 C CNN
+F 2 "Capacitor_THT:CP_Radial_D6.3mm_P2.50mm" H 4938 2550 50  0001 C CNN
 F 3 "" H 4900 2700 50  0001 C CNN
 	1    4900 2700
@@
 	-1   0    0    1
 $EndComp
+Wire Wire Line
+	6450 1950 6450 1800
+Wire Wire Line
+	7500 1950 7500 1900
+NoConn ~ 7400 1950
+Wire Wire Line
+	6450 1800 7500 1800
+NoConn ~ 6350 1950
+NoConn ~ 8850 2750
+Wire Wire Line
+	8450 1950 8450 1800
+Wire Wire Line
+	8450 1800 9050 1800
+Wire Wire Line
+	8550 1950 8550 1900
+Wire Wire Line
+	8550 1900 7500 1900
+Connection ~ 7500 1900
+Wire Wire Line
+	7500 1900 7500 1800
 $EndSCHEMATC

Commit message: last version, too big
Parts:
- added H1, H2, H3, H4: Bolt, KLALIB_Mechanical:Bolt_M3, symbol KLIB_Mechanical:Bolt
Changed lines of the file:
@@
 Wire Wire Line
 	7500 1900 7500 1800
+$Comp
+L KLIB_Mechanical:Bolt H1
+U 1 1 5BA8B8DC
+P 1950 5100
+F 0 "H1" H 2055 5171 50  0000 L CNN
+F 1 "Bolt" H 2055 5080 50  0000 L CNN
+F 2 "KLALIB_Mechanical:Bolt_M3" H 2050 4950 50  0001 L CNN
+F 3 "~" H 2075 5025 50  0001 C CNN
+	1    1950 5100
+	1    0    0    -1
+$EndComp
+$Comp
+L KLIB_Mechanical:Bolt H2
+U 1 1 5BA8B9A4
+P 2300 5100
+F 0 "H2" H 2405 5171 50  0000 L CNN
+F 1 "Bolt" H 2405 5080 50  0000 L CNN
+F 2 "KLALIB_Mechanical:Bolt_M3" H 2400 4950 50  0001 L CNN
+F 3 "~" H 2425 5025 50  0001 C CNN
+	1    2300 5100
+	1    0    0    -1
+$EndComp
+$Comp
+L KLIB_Mechanical:Bolt H3
+U 1 1 5BA8BA08
+P 2650 5100
+F 0 "H3" H 2755 5171 50  0000 L CNN
+F 1 "Bolt" H 2755 5080 50  0000 L CNN
+F 2 "KLALIB_Mechanical:Bolt_M3" H 2750 4950 50  0001 L CNN
+F 3 "~" H 2775 5025 50  0001 C CNN
+	1    2650 5100
+	1    0    0    -1
+$EndComp
+$Comp
+L KLIB_Mechanical:Bolt H4
+U 1 1 5BA8BA77
+P 3000 5100
+F 0 "H4" H 3105 5171 50  0000 L CNN
+F 1 "Bolt" H 3105 5080 50  0000 L CNN
+F 2 "KLALIB_Mechanical:Bolt_M3" H 3100 4950 50  0001 L CNN
+F 3 "~" H 3125 5025 50  0001 C CNN
+	1    3000 5100
+	1    0    0    -1
+$EndComp
 $EndSCHEMATC
