File: adc_7seg_v0.sch (KiCad schematic (older format))
At the start: 34 parts, among them J1 IN, J2 DC, Q1 BC847, U1 MC78M09C, U2 ICL7106, U3 TDSR1350, U4 TDSR1350, U5 TDSR1350

Commit message: first back up
Parts:
- U2: footprint Package_QFP:LQFP-44_10x10mm_P0.8mm -> Package_QFP:TQFP-44_10x10mm_P0.8mm
- U3, U4, U5: footprint KLALIB_Display_7Segment:TDSR1350 -> KLALIB_Display_7Segment:TDSR1350_small_pads
Changed lines of the file:
@@
 F 0 "U3" H 6600 2750 50  0000 L CNN
 F 1 "TDSR1350" H 6500 2650 50  0000 L CNN
-F 2 "KLALIB_Display_7Segment:TDSR1350" H 6800 2050 50  0001 L CNN
+F 2 "KLALIB_Display_7Segment:TDSR1350_small_pads" H 6800 2050 50  0001 L CNN
 F 3 "https://www.vishay.com/docs/85180/tdsr1350.pdf" H 6350 2340 50  0001 L CNN
 	1    6350 2350
@@
 F 0 "U2" H 5450 5350 50  0000 C CNN
 F 1 "ICL7106" H 5450 5250 50  0000 C CNN
-F 2 "Package_QFP:LQFP-44_10x10mm_P0.8mm" H 5200 4150 50  0001 C CNN
+F 2 "Package_QFP:TQFP-44_10x10mm_P0.8mm" H 5200 4150 50  0001 C CNN
 F 3 "https://www.intersil.com/content/dam/Intersil/documents/icl7/icl7106-07-07s.pdf" H 5000 2400 50  0001 C CNN
 	1    5200 4150
@@
 F 0 "U4" H 7650 2750 50  0000 L CNN
 F 1 "TDSR1350" H 7550 2650 50  0000 L CNN
-F 2 "KLALIB_Display_7Segment:TDSR1350" H 7850 2050 50  0001 L CNN
+F 2 "KLALIB_Display_7Segment:TDSR1350_small_pads" H 7850 2050 50  0001 L CNN
 F 3 "https://www.vishay.com/docs/85180/tdsr1350.pdf" H 7400 2340 50  0001 L CNN
 	1    7400 2350
@@
 F 0 "U5" H 8700 2750 50  0000 L CNN
 F 1 "TDSR1350" H 8600 2650 50  0000 L CNN
-F 2 "KLALIB_Display_7Segment:TDSR1350" H 8900 2050 50  0001 L CNN
+F 2 "KLALIB_Display_7Segment:TDSR1350_small_pads" H 8900 2050 50  0001 L CNN
 F 3 "https://www.vishay.com/docs/85180/tdsr1350.pdf" H 8450 2340 50  0001 L CNN
 	1    8450 2350

Commit message: almost last version 0.2.2
Parts:
- removed C4: 100u, Capacitor_THT:CP_Radial_D8.0mm_P3.50mm, symbol Device:CP
- JP1, JP2, JP3: footprint Jumper:SolderJumper-2_P1.3mm_Open_Pad1.0x1.5mm -> KLIB_Mechanical:Jumper
- RV1: footprint KLALIB_Potenciometer_SMD:Potentiometer_Bourns_3269P_Horizontal -> KLALIB_Potenciometer_SMD:Potentiometer_SRPASSIVES_1801
Changed lines of the file:
@@
 F 0 "RV1" H 4430 4496 50  0000 R CNN
 F 1 "5k" H 4430 4405 50  0000 R CNN
-F 2 "KLALIB_Potenciometer_SMD:Potentiometer_Bourns_3269P_Horizontal" H 4500 4450 50  0001 C CNN
+F 2 "KLALIB_Potenciometer_SMD:Potentiometer_SRPASSIVES_1801" H 4500 4450 50  0001 C CNN
 F 3 "" H 4500 4450 50  0001 C CNN
 	1    4500 4450
@@
 F 0 "JP1" H 3100 2755 50  0000 C CNN
 F 1 "2V" H 3100 2664 50  0000 C CNN
-F 2 "Jumper:SolderJumper-2_P1.3mm_Open_Pad1.0x1.5mm" H 3100 2550 50  0001 C CNN
+F 2 "KLIB_Mechanical:Jumper" H 3100 2550 50  0001 C CNN
 F 3 "~" H 3100 2550 50  0001 C CNN
 	1    3100 2550
@@
 F 0 "JP2" H 3100 3355 50  0000 C CNN
 F 1 "20V" H 3100 3264 50  0000 C CNN
-F 2 "Jumper:SolderJumper-2_P1.3mm_Open_Pad1.0x1.5mm" H 3100 3150 50  0001 C CNN
+F 2 "KLIB_Mechanical:Jumper" H 3100 3150 50  0001 C CNN
 F 3 "~" H 3100 3150 50  0001 C CNN
 	1    3100 3150
@@
 F 0 "JP3" H 3100 3655 50  0000 C CNN
 F 1 "200V" H 3100 3564 50  0000 C CNN
-F 2 "Jumper:SolderJumper-2_P1.3mm_Open_Pad1.0x1.5mm" H 3100 3450 50  0001 C CNN
+F 2 "KLIB_Mechanical:Jumper" H 3100 3450 50  0001 C CNN
 F 3 "~" H 3100 3450 50  0001 C CNN
 	1    3100 3450
@@
 $EndComp
 $Comp
-L Device:CP C4
-U 1 1 5BBA66F5
-P 4900 2700
-F 0 "C4" H 5018 2746 50  0000 L CNN
-F 1 "100u" H 5018 2655 50  0000 L CNN
-F 2 "Capacitor_THT:CP_Radial_D8.0mm_P3.50mm" H 4938 2550 50  0001 C CNN
-F 3 "" H 4900 2700 50  0001 C CNN
-	1    4900 2700
-	1    0    0    -1
-$EndComp
-$Comp
 L Device:C C3
 U 1 1 5BBA687B
@@
 $EndComp
 Wire Wire Line
-	5250 2550 4900 2550
-Wire Wire Line
-	4900 2550 4450 2550
-Connection ~ 4900 2550
-Wire Wire Line
 	5250 2550 5250 3000
 Connection ~ 5250 2550
-$Comp
-L power:GND #PWR0111
-U 1 1 5BBB44C2
-P 4900 2850
-F 0 "#PWR0111" H 4900 2600 50  0001 C CNN
-F 1 "GND" H 4905 2677 50  0000 C CNN
-F 2 "" H 4900 2850 50  0001 C CNN
-F 3 "" H 4900 2850 50  0001 C CNN
-	1    4900 2850
-	1    0    0    -1
-$EndComp
 $Comp
 L power:GND #PWR0112
@@
 	-1   0    0    1
 $EndComp
+Wire Wire Line
+	4450 2550 5250 2550
 $EndSCHEMATC
