File: adc_7seg_v0.sch (KiCad schematic (older format))
At the start: 34 parts, among them J1 IN, J2 DC, Q1 BC847, U1 MC78M09C, U2 ICL7106, U3 TDSR1350, U4 TDSR1350, U5 TDSR1350

Commit message: almost last  version
Parts:
- removed C4: 100u, Capacitor_THT:CP_Radial_D8.0mm_P3.50mm, symbol Device:CP
- added H1, H2, H3, H4: Bolt, KLALIB_Mechanical:Bolt_M3, symbol KLIB_Mechanical:Bolt
Connections:
- net at Q1.2 (E), U3.3 (CA): no longer U4.3 (CA), U5.3 (CA)
- net at U3.8 (CA): now also U4.8 (CA), U5.8 (CA)
- no-connect marks 3 -> 6
Other:
- moved on the sheet: C3
Changed lines of the file:
@@
 Wire Wire Line
 	5700 5200 6550 5200
-Wire Wire Line
-	6350 1950 6350 1800
 $Comp
 L Device:R R13
@@
 	1    0    0    -1
 $EndComp
-Wire Wire Line
-	7400 1950 7400 1800
-Wire Wire Line
-	8450 1950 8450 1800
 $Comp
 L KLALIB_Analog_ADC:ICL7106 U2
@@
 	3250 3450 3400 3450
 Wire Wire Line
-	6350 1800 7400 1800
-Wire Wire Line
-	8450 1800 7400 1800
-Connection ~ 7400 1800
-Wire Wire Line
-	8450 1800 9050 1800
-Wire Wire Line
-	9050 1800 9050 5900
-Wire Wire Line
 	9050 5900 6250 5900
-Connection ~ 8450 1800
 NoConn ~ 5700 5300
 NoConn ~ 5700 5400
@@
 $EndComp
 $Comp
-L Device:CP C4
-U 1 1 5BBA66F5
-P 4900 2700
-F 0 "C4" H 5018 2746 50  0000 L CNN
-F 1 "100u" H 5018 2655 50  0000 L CNN
-F 2 "Capacitor_THT:CP_Radial_D8.0mm_P3.50mm" H 4938 2550 50  0001 C CNN
-F 3 "" H 4900 2700 50  0001 C CNN
-	1    4900 2700
-	1    0    0    -1
-$EndComp
-$Comp
 L Device:C C3
 U 1 1 5BBA687B
-P 4450 2700
-F 0 "C3" H 4565 2746 50  0000 L CNN
-F 1 "100n" H 4565 2655 50  0000 L CNN
-F 2 "Capacitor_SMD:C_0603_1608Metric" H 4488 2550 50  0001 C CNN
-F 3 "~" H 4450 2700 50  0001 C CNN
-	1    4450 2700
-	1    0    0    -1
-$EndComp
-Wire Wire Line
-	5250 2550 4900 2550
-Wire Wire Line
-	4900 2550 4450 2550
-Connection ~ 4900 2550
+P 4850 2700
+F 0 "C3" H 4965 2746 50  0000 L CNN
+F 1 "100n" H 4965 2655 50  0000 L CNN
+F 2 "Capacitor_SMD:C_0603_1608Metric" H 4888 2550 50  0001 C CNN
+F 3 "~" H 4850 2700 50  0001 C CNN
+	1    4850 2700
+	1    0    0    -1
+$EndComp
 Wire Wire Line
 	5250 2550 5250 3000
 Connection ~ 5250 2550
 $Comp
-L power:GND #PWR0111
-U 1 1 5BBB44C2
-P 4900 2850
-F 0 "#PWR0111" H 4900 2600 50  0001 C CNN
-F 1 "GND" H 4905 2677 50  0000 C CNN
-F 2 "" H 4900 2850 50  0001 C CNN
-F 3 "" H 4900 2850 50  0001 C CNN
-	1    4900 2850
-	1    0    0    -1
-$EndComp
-$Comp
 L power:GND #PWR0112
 U 1 1 5BBB4518
-P 4450 2850
-F 0 "#PWR0112" H 4450 2600 50  0001 C CNN
-F 1 "GND" H 4455 2677 50  0000 C CNN
-F 2 "" H 4450 2850 50  0001 C CNN
-F 3 "" H 4450 2850 50  0001 C CNN
-	1    4450 2850
+P 4850 2850
+F 0 "#PWR0112" H 4850 2600 50  0001 C CNN
+F 1 "GND" H 4855 2677 50  0000 C CNN
+F 2 "" H 4850 2850 50  0001 C CNN
+F 3 "" H 4850 2850 50  0001 C CNN
+	1    4850 2850
 	1    0    0    -1
 $EndComp
@@
 	-1   0    0    1
 $EndComp
+Wire Wire Line
+	4850 2550 5250 2550
+$Comp
+L KLIB_Mechanical:Bolt H1
+U 1 1 5BAAF32B
+P 2000 5150
+F 0 "H1" H 2105 5221 50  0000 L CNN
+F 1 "Bolt" H 2105 5130 50  0000 L CNN
+F 2 "KLALIB_Mechanical:Bolt_M3" H 2100 5000 50  0001 L CNN
+F 3 "~" H 2125 5075 50  0001 C CNN
+	1    2000 5150
+	1    0    0    -1
+$EndComp
+$Comp
+L KLIB_Mechanical:Bolt H2
+U 1 1 5BAAF48D
+P 2400 5150
+F 0 "H2" H 2505 5221 50  0000 L CNN
+F 1 "Bolt" H 2505 5130 50  0000 L CNN
+F 2 "KLALIB_Mechanical:Bolt_M3" H 2500 5000 50  0001 L CNN
+F 3 "~" H 2525 5075 50  0001 C CNN
+	1    2400 5150
+	1    0    0    -1
+$EndComp
+$Comp
+L KLIB_Mechanical:Bolt H3
+U 1 1 5BAAF52F
+P 2800 5150
+F 0 "H3" H 2905 5221 50  0000 L CNN
+F 1 "Bolt" H 2905 5130 50  0000 L CNN
+F 2 "KLALIB_Mechanical:Bolt_M3" H 2900 5000 50  0001 L CNN
+F 3 "~" H 2925 5075 50  0001 C CNN
+	1    2800 5150
+	1    0    0    -1
+$EndComp
+$Comp
+L KLIB_Mechanical:Bolt H4
+U 1 1 5BAAF58C
+P 3200 5150
+F 0 "H4" H 3305 5221 50  0000 L CNN
+F 1 "Bolt" H 3305 5130 50  0000 L CNN
+F 2 "KLALIB_Mechanical:Bolt_M3" H 3300 5000 50  0001 L CNN
+F 3 "~" H 3325 5075 50  0001 C CNN
+	1    3200 5150
+	1    0    0    -1
+$EndComp
+NoConn ~ 8450 1950
+NoConn ~ 7400 1950
+Wire Wire Line
+	6450 1950 6450 1800
+Wire Wire Line
+	9050 1650 6350 1650
+Wire Wire Line
+	9050 1650 9050 5900
+Wire Wire Line
+	6350 1650 6350 1950
+Wire Wire Line
+	8550 1800 8550 1950
+$Comp
+L power:PWR_FLAG #FLG0101
+U 1 1 5BB0563B
+P 2300 1850
+F 0 "#FLG0101" H 2300 1925 50  0001 C CNN
+F 1 "PWR_FLAG" V 2300 1978 50  0001 L CNN
+F 2 "" H 2300 1850 50  0001 C CNN
+F 3 "~" H 2300 1850 50  0001 C CNN
+	1    2300 1850
+	0    1    1    0
+$EndComp
+Connection ~ 2300 1850
+$Comp
+L power:PWR_FLAG #FLG0102
+U 1 1 5BB0C8D1
+P 4250 5150
+F 0 "#FLG0102" H 4250 5225 50  0001 C CNN
+F 1 "PWR_FLAG" V 4250 5278 50  0001 L CNN
+F 2 "" H 4250 5150 50  0001 C CNN
+F 3 "~" H 4250 5150 50  0001 C CNN
+	1    4250 5150
+	0    -1   -1   0
+$EndComp
+Connection ~ 4250 5150
+$Comp
+L power:PWR_FLAG #FLG0103
+U 1 1 5BB1030C
+P 4800 5300
+F 0 "#FLG0103" H 4800 5375 50  0001 C CNN
+F 1 "PWR_FLAG" V 4800 5428 50  0001 L CNN
+F 2 "" H 4800 5300 50  0001 C CNN
+F 3 "~" H 4800 5300 50  0001 C CNN
+	1    4800 5300
+	0    -1   -1   0
+$EndComp
+Connection ~ 4800 5300
+Wire Wire Line
+	7500 1800 8550 1800
+Wire Wire Line
+	6450 1800 7500 1800
+Connection ~ 7500 1800
+Wire Wire Line
+	7500 1950 7500 1800
+NoConn ~ 8850 2750
 $EndSCHEMATC

Commit message: last
Connections:
- net at U3.8 (CA), U4.8 (CA): no longer U5.8 (CA)
- net at U4.3 (CA): now also U5.3 (CA)
- no-connect marks 6 -> 5
Changed lines of the file:
@@
 	1    0    0    -1
 $EndComp
-NoConn ~ 8450 1950
 NoConn ~ 7400 1950
 Wire Wire Line
@@
 Wire Wire Line
 	6350 1650 6350 1950
-Wire Wire Line
-	8550 1800 8550 1950
 $Comp
 L power:PWR_FLAG #FLG0101
@@
 Connection ~ 4800 5300
 Wire Wire Line
-	7500 1800 8550 1800
-Wire Wire Line
 	6450 1800 7500 1800
-Connection ~ 7500 1800
 Wire Wire Line
 	7500 1950 7500 1800
 NoConn ~ 8850 2750
+Wire Wire Line
+	8450 1950 8450 1850
+Wire Wire Line
+	7400 1950 7400 1850
+Wire Wire Line
+	7400 1850 8450 1850
 $EndSCHEMATC
